File: MarineBoard/MarineBoard.kicad_sch (KiCad schematic)
At the start: 149 parts, among them CN1 MKDSN 1,5/ 2-5,08, CN2 MKDSN 1,5/ 2-5,08, CN3 SM04B-SRSS-TB (LF)(SN), J1 USB_C_Receptacle_USB2.0_16P, J3 Conn_02x09_Top_Bottom, Q1 IPL60R075CFD7, Q2 S8050, Q3 S8050, U1 SY8089A1AAC, U10 PC817C-S, U11 SN65HVD230DR, U12 DB125-3.5-3P-GN-S, U13 DB125-3.5-3P-GN-S, U14 PC817C-S, U15 TC4427EPA, U16 PC817C-S, U17 PC817C-S, U18 INA226, U19 INA226, U2 INA226, U3 TPS5430DDA, U4 DB125-3.5-2P-GN-S, U5 DB125-3.5-2P-GN-S, U6 DB125-3.5-2P-GN-S, U7 DB125-3.5-3P-GN-S, U8 ESP32-S3-WROOM-2-N32R16V, U9 DB125-3.5-3P-GN-S

Commit message: MarineBoard: update KiCad project + add EasyEDA library assets
- Update PCB, schematic, project, and library-table files
- Add EasyEDA symbol/footprint/3D-model assets (C0402, C1210, R2512, SMA)
- Add new documentation images (ESP32, FSPI, RPM)

Co-Authored-By: Claude Sonnet 5 <noreply@anthropic.com>
Parts:
- removed R16: 1K, Resistor_SMD:R_0402_1005Metric, symbol Device:R
- added C33: 1.2uF 100V, Capacitor_SMD:C_1210_3225Metric, symbol EasyEDA:HGC0402R5105K500NTEJ
- added R37: 100K, easyeda2kicad:R0805, symbol easyeda2kicad:0805W8F1003T5E_C149504
- added R45: 2K2, EasyEDA:R2512, symbol EasyEDA:CRGP2512F2K2
- added U20: SMAJ6.8CA, EasyEDA:SMA_L4.4-W2.6-LS5.0-BI, symbol EasyEDA:SMAJ6.8CA_C3001958
Connections:
- net RPM is gone; now on net SH+: U13.2
- net GND: now also R37.1, U20.2 (A)
- net SH+: now also C33.1
- net at D8.2 (K), U10.1: now also R45.2, U20.1 (K)
- new net: C33.2, R37.2, R45.1
Other:
- note added: "NEW"
- note added: "RPM input"
- moved on the sheet: D12, D8, R17, R18, R22, R23, R26, U10, U14
