File: MarineBoard/MarineBoard.kicad_sch (KiCad schematic)
At the start: 152 parts, among them CN1 MKDSN 1,5/ 2-5,08, CN2 MKDSN 1,5/ 2-5,08, CN3 SM04B-SRSS-TB (LF)(SN), J1 USB_C_Receptacle_USB2.0_16P, J3 Conn_02x09_Top_Bottom, Q1 IPL60R075CFD7, Q2 S8050, Q3 S8050, U1 SY8089A1AAC, U10 PC817C-S, U11 SN65HVD230DR, U12 DB125-3.5-3P-GN-S, U13 DB125-3.5-3P-GN-S, U14 PC817C-S, U15 TC4427EPA, U16 PC817C-S, U17 PC817C-S, U18 INA226, U19 INA226, U2 INA226, U20 SMAJ6.8CA, U3 TPS5430DDA, U4 DB125-3.5-2P-GN-S, U5 DB125-3.5-2P-GN-S, U6 DB125-3.5-2P-GN-S, U7 DB125-3.5-3P-GN-S, U8 ESP32-S3-WROOM-2-N32R16V, U9 DB125-3.5-3P-GN-S

Commit message: MarineBoard: consolidate LCSC libraries into EasyEDA (#96)
Merge 0623, easyeda2kicad, and root EasyEDA.pretty into Lib/EasyEDA.
Retarget schematic/PCB nicknames and 3D paths to the project library.
Import Hirose FH12-18S QSPI symbol and footprint; J3 on the board is unchanged.
Parts:
- C20: footprint easyeda2kicad:CAP-SMD_BD6.3-L6.6-W6.6-FD -> EasyEDA:CAP-SMD_BD6.3-L6.6-W6.6-FD; symbol easyeda2kicad:RVT1A221M0605-C72494 -> EasyEDA:RVT1A221M0605-C72494
- C4, C8: symbol easyeda2kicad:CL21A226MAYNNNE -> EasyEDA:CL21A226MAYNNNE
- C6: symbol easyeda2kicad:0603CG6R8C500NT -> EasyEDA:0603CG6R8C500NT
- CN1, CN2: footprint easyeda2kicad:CONN-TH_2P-P5.08_1729128 -> EasyEDA:CONN-TH_2P-P5.08_1729128
- CN3: footprint easyeda2kicad:CONN-SMD_4P-P1.00_SM04B-SRSS-TB-LF-SN -> EasyEDA:CONN-SMD_4P-P1.00_SM04B-SRSS-TB-LF-SN
- D2, D3: footprint 0623:SOD-882_L1.0-W0.6-BI -> EasyEDA:SOD-882_L1.0-W0.6-BI
- D5: footprint easyeda2kicad:SMC_L7.1-W6.2-LS8.1-RD -> EasyEDA:SMC_L7.1-W6.2-LS8.1-RD
- J1: footprint 0623:USB_C_Receptacle_HCTL_HC-TYPE-C-16P-01A -> EasyEDA:USB_C_Receptacle_HCTL_HC-TYPE-C-16P-01A
- L1: footprint easyeda2kicad:L2520 -> EasyEDA:L2520; symbol easyeda2kicad:DFE252012F-1R0M=P2 -> EasyEDA:DFE252012F-1R0M=P2
- L10, L7, L9: symbol L0805:BLM21PG331SN1D -> EasyEDA:BLM21PG331SN1D
- L3, L4, L6: footprint 0623:L0805 -> EasyEDA:L0805
- Q2, Q3: footprint 0623:SOT-23-3_L2.9-W1.3-P1.90-LS2.3-BR -> EasyEDA:SOT-23-3_L2.9-W1.3-P1.90-LS2.3-BR
- R37, R4: footprint easyeda2kicad:R0805 -> EasyEDA:R0805; symbol easyeda2kicad:0805W8F1003T5E_C149504 -> EasyEDA:0805W8F1003T5E_C149504
- R8: footprint easyeda2kicad:R0805 -> EasyEDA:R0805; symbol easyeda2kicad:0805W8F2202T5E -> EasyEDA:0805W8F2202T5E
- U1: footprint easyeda2kicad:TSOT-23-5_L2.9-W1.6-P0.95-LS2.8-BR -> EasyEDA:TSOT-23-5_L2.9-W1.6-P0.95-LS2.8-BR; symbol easyeda2kicad:SY8089A1AAC -> EasyEDA:SY8089A1AAC
- U18, U19: footprint 0623:VSSOP-10_3x3mm_P0.5mm -> EasyEDA:VSSOP-10_3x3mm_P0.5mm
Changed lines of the file:
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@@
 			)
 		)
-		(property "Footprint" "0623:SOT-23-3_L2.9-W1.3-P1.90-LS2.3-BR"
+		(property "Footprint" "EasyEDA:SOT-23-3_L2.9-W1.3-P1.90-LS2.3-BR"
 			(at 421.64 241.3 0)
 			(hide yes)
@@
 			)
 		)
-		(property "Footprint" "0623:SOD-882_L1.0-W0.6-BI"
+		(property "Footprint" "EasyEDA:SOD-882_L1.0-W0.6-BI"
 			(at 95.25 52.07 0)
 			(hide yes)
@@
 	)
 	(symbol
-		(lib_id "easyeda2kicad:0603CG6R8C500NT")
+		(lib_id "EasyEDA:0603CG6R8C500NT")
 		(at 275.59 38.1 90)
 		(unit 1)
@@
 	)
 	(symbol
-		(lib_id "easyeda2kicad:0805W8F1003T5E_C149504")
+		(lib_id "EasyEDA:0805W8F1003T5E_C149504")
 		(at 176.53 179.07 90)
 		(unit 1)
@@
 			)
 		)
-		(property "Footprint" "easyeda2kicad:R0805"
+		(property "Footprint" "EasyEDA:R0805"
 			(at 184.15 179.07 0)
 			(hide yes)
@@
 			)
 		)
-		(property "Footprint" "0623:SOT-23-3_L2.9-W1.3-P1.90-LS2.3-BR"
+		(property "Footprint" "EasyEDA:SOT-23-3_L2.9-W1.3-P1.90-LS2.3-BR"
 			(at 330.2 274.32 0)
 			(hide yes)
@@
 			)
 		)
-		(property "Footprint" "0623:VSSOP-10_3x3mm_P0.5mm"
+		(property "Footprint" "EasyEDA:VSSOP-10_3x3mm_P0.5mm"
 			(at 85.09 266.7 0)
 			(hide yes)
@@
 	)
 	(symbol
-		(lib_id "easyeda2kicad:DFE252012F-1R0M=P2")
+		(lib_id "EasyEDA:DFE252012F-1R0M=P2")
 		(at 264.16 33.02 0)
 		(unit 1)
@@
 			)
 		)
-		(property "Footprint" "easyeda2kicad:L2520"
+		(property "Footprint" "EasyEDA:L2520"
 			(at 264.16 40.64 0)
 			(hide yes)
@@
 	)
 	(symbol
-		(lib_id "easyeda2kicad:0805W8F1003T5E_C149504")
+		(lib_id "EasyEDA:0805W8F1003T5E_C149504")
 		(at 270.51 39.37 90)
 		(unit 1)
@@
 			)
 		)
-		(property "Footprint" "easyeda2kicad:R0805"
+		(property "Footprint" "EasyEDA:R0805"
 			(at 278.13 39.37 0)
 			(hide yes)
@@
 	(symbol
 		(lib_name "BLM21PG331SN1D_2")
-		(lib_id "L0805:BLM21PG331SN1D")
+		(lib_id "EasyEDA:BLM21PG331SN1D")
 		(at 125.73 241.3 0)
 		(unit 1)
@@
 			)
 		)
-		(property "Footprint" "easyeda2kicad:CONN-TH_2P-P5.08_1729128"
+		(property "Footprint" "EasyEDA:CONN-TH_2P-P5.08_1729128"
 			(at 425.45 33.02 0)
 			(hide yes)
@@
 	(symbol
 		(lib_name "BLM21PG331SN1D_2")
-		(lib_id "L0805:BLM21PG331SN1D")
+		(lib_id "EasyEDA:BLM21PG331SN1D")
 		(at 325.12 124.46 90)
 		(unit 1)
@@
 			)
 		)
-		(property "Footprint" "easyeda2kicad:CONN-SMD_4P-P1.00_SM04B-SRSS-TB-LF-SN"
+		(property "Footprint" "EasyEDA:CONN-SMD_4P-P1.00_SM04B-SRSS-TB-LF-SN"
 			(at 433.07 91.44 0)
 			(hide yes)
@@
 	(symbol
 		(lib_name "BLM21PG331SN1D_2")
-		(lib_id "L0805:BLM21PG331SN1D")
+		(lib_id "EasyEDA:BLM21PG331SN1D")
 		(at 43.18 241.3 0)
 		(unit 1)
@@
 	)
 	(symbol
-		(lib_id "easyeda2kicad:SY8089A1AAC")
+		(lib_id "EasyEDA:SY8089A1AAC")
 		(at 248.92 35.56 0)
 		(unit 1)
@@
 			)
 		)
-		(property "Footprint" "easyeda2kicad:TSOT-23-5_L2.9-W1.6-P0.95-LS2.8-BR"
+		(property "Footprint" "EasyEDA:TSOT-23-5_L2.9-W1.6-P0.95-LS2.8-BR"
 			(at 248.92 45.72 0)
 			(hide yes)
@@
 			)
 		)
-		(property "Footprint" "0623:L0805"
+		(property "Footprint" "EasyEDA:L0805"
 			(at 203.2 96.52 0)
 			(hide yes)
@@
 	)
 	(symbol
-		(lib_id "easyeda2kicad:CL21A226MAYNNNE")
+		(lib_id "EasyEDA:CL21A226MAYNNNE")
 		(at 283.21 46.99 90)
 		(unit 1)
@@
 			)
 		)
-		(property "Footprint" "easyeda2kicad:CONN-TH_2P-P5.08_1729128"
+		(property "Footprint" "EasyEDA:CONN-TH_2P-P5.08_1729128"
 			(at 425.45 40.64 0)
 			(hide yes)
@@
 			)
 		)
-		(property "Footprint" "0623:VSSOP-10_3x3mm_P0.5mm"
+		(property "Footprint" "EasyEDA:VSSOP-10_3x3mm_P0.5mm"
 			(at 162.56 266.7 0)
 			(hide yes)
@@
 			)
 		)
-		(property "Footprint" "0623:USB_C_Receptacle_HCTL_HC-TYPE-C-16P-01A"
+		(property "Footprint" "EasyEDA:USB_C_Receptacle_HCTL_HC-TYPE-C-16P-01A"
 			(at 71.12 39.37 0)
 			(hide yes)
@@
 			)
 		)
-		(property "Footprint" "0623:L0805"
+		(property "Footprint" "EasyEDA:L0805"
 			(at 110.49 77.47 0)
 			(hide yes)
@@
 	)
 	(symbol
-		(lib_id "easyeda2kicad:CL21A226MAYNNNE")
+		(lib_id "EasyEDA:CL21A226MAYNNNE")
 		(at 224.79 46.99 90)
 		(unit 1)
@@
 	)
 	(symbol
-		(lib_id "easyeda2kicad:0805W8F2202T5E")
+		(lib_id "EasyEDA:0805W8F2202T5E")
 		(at 270.51 49.53 90)
 		(unit 1)
@@
 			)
 		)
-		(property "Footprint" "easyeda2kicad:R0805"
+		(property "Footprint" "EasyEDA:R0805"
 			(at 278.13 49.53 0)
 			(hide yes)
@@
 			)
 		)
-		(property "Footprint" "0623:L0805"
+		(property "Footprint" "EasyEDA:L0805"
 			(at 69.85 77.47 0)
 			(hide yes)
@@
 			)
 		)
-		(property "Footprint" "0623:SOD-882_L1.0-W0.6-BI"
+		(property "Footprint" "EasyEDA:SOD-882_L1.0-W0.6-BI"
 			(at 95.25 33.02 0)
 			(hide yes)
@@
 			)
 		)
-		(property "Footprint" "easyeda2kicad:SMC_L7.1-W6.2-LS8.1-RD"
+		(property "Footprint" "EasyEDA:SMC_L7.1-W6.2-LS8.1-RD"
 			(at 39.37 69.85 0)
 			(hide yes)
@@
 	)
 	(symbol
-		(lib_id "easyeda2kicad:RVT1A221M0605-C72494")
+		(lib_id "EasyEDA:RVT1A221M0605-C72494")
 		(at 170.18 104.14 0)
 		(unit 1)
@@
 			)
 		)
-		(property "Footprint" "easyeda2kicad:CAP-SMD_BD6.3-L6.6-W6.6-FD"
+		(property "Footprint" "EasyEDA:CAP-SMD_BD6.3-L6.6-W6.6-FD"
 			(at 170.18 115.57 0)
 			(hide yes)
