File: MarineBoard/MarineBoard.kicad_pcb (KiCad board)
At the start: 4 copper layers, 66.5 x 70 mm, 151 parts, among them CN1 MKDSN 1,5/ 2-5,08, CN2 MKDSN 1,5/ 2-5,08, CN3 SM04B-SRSS-TB (LF)(SN), J1 USB_C_Receptacle_USB2.0_16P, J3 Conn_02x09_Top_Bottom, Q1 IPL60R075CFD7, Q2 S8050, Q3 S8050, U1 SY8089A1AAC, U10 PC817C-S, U11 SN65HVD230DR, U12 DB125-3.5-3P-GN-S, U13 DB125-3.5-3P-GN-S, U14 PC817C-S, U15 TC4427EPA, U16 PC817C-S, U17 PC817C-S, U18 INA226, U19 INA226, U2 INA226, U20 SMAJ6.8CA, U3 TPS5430DDA, U4 DB125-3.5-2P-GN-S, U5 DB125-3.5-2P-GN-S, U6 DB125-3.5-2P-GN-S, U7 DB125-3.5-3P-GN-S, U8 ESP32-S3-WROOM-2-N32R16V, U9 DB125-3.5-3P-GN-S

Commit message: MarineBoard: consolidate LCSC libraries into EasyEDA (#96)
Merge 0623, easyeda2kicad, and root EasyEDA.pretty into Lib/EasyEDA.
Retarget schematic/PCB nicknames and 3D paths to the project library.
Import Hirose FH12-18S QSPI symbol and footprint; J3 on the board is unchanged.
Parts:
- C20: footprint easyeda2kicad:CAP-SMD_BD6.3-L6.6-W6.6-FD -> EasyEDA:CAP-SMD_BD6.3-L6.6-W6.6-FD
- CN1, CN2: footprint easyeda2kicad:CONN-TH_2P-P5.08_1729128 -> EasyEDA:CONN-TH_2P-P5.08_1729128
- CN3: footprint easyeda2kicad:CONN-SMD_4P-P1.00_SM04B-SRSS-TB-LF-SN -> EasyEDA:CONN-SMD_4P-P1.00_SM04B-SRSS-TB-LF-SN
- D2, D3: footprint 0623:SOD-882_L1.0-W0.6-BI -> EasyEDA:SOD-882_L1.0-W0.6-BI
- D5: footprint easyeda2kicad:SMC_L7.1-W6.2-LS8.1-RD -> EasyEDA:SMC_L7.1-W6.2-LS8.1-RD
- J1: footprint 0623:USB_C_Receptacle_HCTL_HC-TYPE-C-16P-01A -> EasyEDA:USB_C_Receptacle_HCTL_HC-TYPE-C-16P-01A
- L1: footprint easyeda2kicad:L2520 -> EasyEDA:L2520
- L3, L4, L6: footprint 0623:L0805 -> EasyEDA:L0805
- Q2, Q3: footprint 0623:SOT-23-3_L2.9-W1.3-P1.90-LS2.3-BR -> EasyEDA:SOT-23-3_L2.9-W1.3-P1.90-LS2.3-BR
- R37, R4, R8: footprint easyeda2kicad:R0805 -> EasyEDA:R0805
- U1: footprint easyeda2kicad:TSOT-23-5_L2.9-W1.6-P0.95-LS2.8-BR -> EasyEDA:TSOT-23-5_L2.9-W1.6-P0.95-LS2.8-BR
- U18, U19: footprint 0623:VSSOP-10_3x3mm_P0.5mm -> EasyEDA:VSSOP-10_3x3mm_P0.5mm
