File: MarineBoard/MarineBoard.kicad_pcb (KiCad board)
At the start: 4 copper layers, 83 x 67.5 mm, 162 parts, among them CN1 MKDSN 1,5/ 2-5,08, CN2 MKDSN 1,5/ 2-5,08, CN3 SM04B-SRSS-TB (LF)(SN), CN4 BM10B-GHS-TBT, J1 USB_C_Receptacle_USB2.0_16P, Q2 S8050, Q3 S8050, Q4 BUK762R4-60E, U1 SY8089A1AAC, U11 SN65HVD230DR, U12 DB125-3.5-3P-GN-S, U13 DB125-3.5-3P-GN-S, U14 PC817C-S, U16 PC817C-S, U17 PC817C-S, U18 INA226, U19 INA226, U2 INA226, U21 PC817C-S, U22 SN74LVC1G14DBVR, U23 MCP1407-E/MF_C640313, U3 TPS5430DDA, U4 DB125-3.5-2P-GN-S, U5 DB125-3.5-2P-GN-S, U6 DB125-3.5-2P-GN-S, U7 DB125-3.5-3P-GN-S, U8 ESP32-S3-WROOM-2-N32R16V, U9 DB125-3.5-3P-GN-S

Commit message: MarineBoard: enclosure, PCBWay delivery, 5-unit BOM (#194)
Enclosure: printed PA12 box 129.4 x 107.9 x 44 mm, built by a parametric
FreeCAD script (enclosure/make_enclosure.py; fit_board.py checks the KiCad
board STEP against it). IP67 panel connectors with engraved legends
(EW-LP20 power/PWM, M12-5 CAN, 12G for TMP/RPM/ENBL, relay, shunt,
levels), 2 mm silicone-cord seal, D5 light pipe, 4 x M3x6 board and
4 x M3x10 lid screws, no USB opening (flash before boxing, then OTA).
STEP + STL exports, FreeCAD docs, render, and the PCBWay print/parts
order sheet. Documented in Technical Specs -> Enclosure; README,
INSTALLATION section 8.3 and Technical Specifications point to it.

Also: PCBWay's 15 Aug delivery package (design files, CAM, the earlier
enclosure, now marked superseded), the connector purchase list, and
the 5-unit assembly BOM. Order numbers are kept out of the file names.
Board BOM: real part numbers for generic parts (BLM21PG331SN1D,
KT-0603R, MCP1407-E/MF); production files regenerated; no copper change.
FreeCAD *.FCBak backups ignored. Project Claude permissions updated.

Signal K plugin configs stay uncommitted (local MQTT credentials).

Co-Authored-By: Claude Opus 5.5 <noreply@anthropic.com>
Parts:
- D16: value LED -> KT-0603R
- L10, L7, L9: value FerriteBead -> BLM21PG331SN1D
- U23: value MCP1407-E/MF_C640313 -> MCP1407-E/MF
