File: MarineBoard/MarineBoard.kicad_pcb (KiCad board)
At the start: 4 copper layers, 83 x 67.5 mm, 162 parts, among them CN1 MKDSN 1,5/ 2-5,08, CN2 MKDSN 1,5/ 2-5,08, CN3 SM04B-SRSS-TB (LF)(SN), CN4 BM10B-GHS-TBT, J1 USB_C_Receptacle_USB2.0_16P, Q2 S8050, Q3 S8050, Q4 BUK762R4-60E, U1 SY8089A1AAC, U11 SN65HVD230DR, U12 DB125-3.5-3P-GN-S, U13 DB125-3.5-3P-GN-S, U14 PC817C-S, U16 PC817C-S, U17 PC817C-S, U18 INA226, U19 INA226, U2 INA226, U21 PC817C-S, U22 SN74LVC1G14DBVR, U23 MCP1407-E/MF, U3 TPS5430DDA, U4 DB125-3.5-2P-GN-S, U5 DB125-3.5-2P-GN-S, U6 DB125-3.5-2P-GN-S, U7 DB125-3.5-3P-GN-S, U8 ESP32-S3-WROOM-2-N32R16V, U9 DB125-3.5-3P-GN-S

Commit message: Answer PCBWay's T-1P19 questions and fit the fuses and shunt
PCBWay inserts the MINI fuses into F1-F4 and fits the 1.27 mm shunt on JP1. F2 is Eaton ATM-1 because Littelfuse 0297001.WXNV is not a real part. Descriptions for D2/D3, D5, D21, R5/R6 and R47 match the replies.

#199
Parts:
- D5: value WS2812B-2020 -> WS2812B-2020-V6
Changed lines of the file:
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@@
 			)
 		)
-		(property "Description" "XF-506P MINI blade fuse holder"
+		(property "Description" "XF-506P MINI blade fuse holder. Insert Littelfuse 0297002.WXNV, 2 A 32 V MINI blade, into this holder."
 			(at 0 0 0)
 			(layer "F.Fab")
@@
 			)
 		)
-		(property "Value" "WS2812B-2020"
+		(property "Value" "WS2812B-2020-V6"
 			(at 0 2.2 0)
 			(layer "F.Fab")
@@
 			)
 		)
-		(property "Description" "RGB LED with integrated controller, 2.0 x 2.0 mm"
+		(property "Description" "RGB LED with integrated controller, Worldsemi WS2812B-2020-V6, 2.0 x 2.0 mm"
 			(at 0 0 0)
 			(unlocked yes)
@@
 			)
 		)
-		(property "MPN" "WS2812B-2020"
+		(property "MPN" "WS2812B-2020-V6"
 			(at 0 0 0)
 			(unlocked yes)
@@
 			)
 		)
-		(property "Description" "1.27 mm 1x2 vertical pin header. Leave open; shunt is supplied loose."
+		(property "Description" "1.27 mm 1x2 vertical pin header. Fit BOOMELE shunt MPN 1.27, LCSC C150949, onto these pins."
 			(at 0 0 0)
 			(layer "F.Fab")
@@
 			)
 		)
-		(property "Description" "XF-506P MINI blade fuse holder"
+		(property "Description" "XF-506P MINI blade fuse holder. Insert Eaton Bussmann ATM-1, 1 A 32 V MINI blade, into this holder."
 			(at 0 0 0)
 			(layer "F.Fab")
@@
 			)
 		)
-		(property "Description" "XF-506P MINI blade fuse holder"
+		(property "Description" "XF-506P MINI blade fuse holder. Insert Littelfuse 0297010.WXNV, 10 A 32 V MINI blade, into this holder."
 			(at 0 0 0)
 			(layer "F.Fab")
@@
 			)
 		)
-		(property "Description" "XF-506P MINI blade fuse holder"
+		(property "Description" "XF-506P MINI blade fuse holder. Insert Littelfuse 0297010.WXNV, 10 A 32 V MINI blade, into this holder."
 			(at 0 0 0)
 			(layer "F.Fab")
@@
 			)
 		)
-		(property "Description" "2.2 kohm +/-1% 1W 2512"
+		(property "Description" "2.2 kohm +/-1% 2W 2512"
 			(at 0 0 0)
 			(layer "B.Fab")
@@
 			)
 		)
-		(property "Description" "75V 150mA switching diode SOD-123; drops D5 VDD ~0.65 V so 3.3 V data meets WS2812B VIH (#183)"
+		(property "Description" "75V 150mA switching diode, SOD-123, Diodes Inc 1N4148W-7-F"
 			(at 0 0 270)
 			(unlocked yes)
@@
 			)
 		)
-		(property "Description" "5V bidirectional ESD diode, DFN1006-2L (SOD-882 land)"
+		(property "Description" "5V bidirectional ESD diode H5VL10B. Manufacturer package DFN1006-2L. Board land is SOD-882, the same 1.0 x 0.6 mm pad."
 			(at 0 0 270)
 			(unlocked yes)
@@
 			)
 		)
-		(property "Description" "5V bidirectional ESD diode, DFN1006-2L (SOD-882 land)"
+		(property "Description" "5V bidirectional ESD diode H5VL10B. Manufacturer package DFN1006-2L. Board land is SOD-882, the same 1.0 x 0.6 mm pad."
 			(at 0 0 270)
 			(unlocked yes)
@@
 			)
 		)
-		(property "Description" "33 ohm +/-5% 0402"
+		(property "Description" "33 ohm +/-1% 0402"
 			(at 0 0 0)
 			(layer "B.Fab")
@@
 			)
 		)
-		(property "Description" "33 ohm +/-5% 0402"
+		(property "Description" "33 ohm +/-1% 0402"
 			(at 0 0 0)
 			(layer "B.Fab")
